Commit message: changed the urdf files to match the deepracer specifications

File: simulation_ws/src/deepracer_simulation/urdf/racecar.xacro (robot description, xacro)
@@ -11,5 +11,5 @@
   </link>
   <joint name="base_link_joint" type="fixed">
-    <origin xyz="0 0 0.05" rpy="0 0 0" />
+    <origin xyz="0 0 0.03" rpy="0 0 0" />
     <parent link="base_link" />
     <child link="chassis" />
@@ -148,6 +148,6 @@
   <link name="zed_camera_link">
     <inertial>
-      <mass value="1e-5" />
-      <origin xyz="0 0 0" rpy="0 -0.26 0"/>
+      <mass value="1e-3" />
+      <origin xyz="0 0 0" rpy="0 0 0"/>
       <inertia ixx="1e-6" ixy="0" ixz="0" iyy="1e-6" iyz="0" izz="1e-6" />
     </inertial>
@@ -167,5 +167,5 @@
   </link>
   <joint name="zed_camera_joint" type="fixed">
-    <origin xyz="0.25 0 0.14" rpy="0 0 0"/>
+    <origin xyz="0.20 0 0.10" rpy="0 0.2731415 0"/>
     <parent link="chassis"/>
     <child link="zed_camera_link"/>
@@ -177,5 +177,5 @@
   <link name="camera_link"><!-- this needs to match the name in zed_wrapper/zed_tf.launch -->
     <inertial>
-      <mass value="1e-5" />
+      <mass value="1e-3" />
       <origin xyz="0 0 0" rpy="0 0 0"/>
       <inertia ixx="1e-6" ixy="0" ixz="0" iyy="1e-6" iyz="0" izz="1e-6" />
@@ -184,11 +184,11 @@
   <link name="zed_camera_right_link">
     <inertial>
-      <mass value="1e-5" />
-      <origin xyz="0 0 0" rpy="0 0 0"/>
+      <mass value="1e-3" />
+      <origin xyz="0 0.005 0" rpy="0 0 0"/>
       <inertia ixx="1e-6" ixy="0" ixz="0" iyy="1e-6" iyz="0" izz="1e-6" />
     </inertial>
   </link>
   <joint name="zed_camera_left_joint" type="fixed">
-    <origin xyz="0 0.06 0" rpy="0 0 0"/>
+    <origin xyz="0 0 0" rpy="0 0 0"/>
     <parent link="zed_camera_link"/>
     <child link="camera_link"/>
@@ -196,5 +196,5 @@
   </joint>
   <joint name="zed_camera_right_joint" type="fixed">
-    <origin xyz="0 -0.06 0" rpy="0 0 0"/>
+    <origin xyz="0 -0 0" rpy="0 0 0"/>
     <parent link="zed_camera_link"/>
     <child link="zed_camera_right_link"/>

Commit message: fixing the -0 typo in racecar xacro

File: simulation_ws/src/deepracer_simulation/urdf/racecar.xacro (robot description, xacro)
@@ -196,5 +196,5 @@
   </joint>
   <joint name="zed_camera_right_joint" type="fixed">
-    <origin xyz="0 -0 0" rpy="0 0 0"/>
+    <origin xyz="0 0 0" rpy="0 0 0"/>
     <parent link="zed_camera_link"/>
     <child link="zed_camera_right_link"/>
